Commit message: Use LeRobot names for actuated URDF joints

File: URDF/LeKiwi.urdf (robot description, URDF)
Before this commit: robot LeKiwi, 45 links, 44 joints
Joints:
- removed joint ST3215_Servo_Motor-v1-1_Revolute-62
- removed joint ST3215_Servo_Motor-v1-2_Revolute-60
- removed joint ST3215_Servo_Motor-v1_Revolute-64
- removed joint STS3215_03a-v1-1_Revolute-49
- removed joint STS3215_03a-v1-2_Revolute-51
- removed joint STS3215_03a-v1-3_Revolute-53
- removed joint STS3215_03a-v1-4_Revolute-57
- removed joint STS3215_03a-v1_Revolute-45
- removed joint STS3215_03a_Wrist_Roll-v1_Revolute-55
- added joint arm_elbow_flex: type continuous, parent STS3215_03a-v1-2, child SO_ARM100_08k_Mirror-v1, origin xyz=0.0346 -0.013069710000000002 0.03178184000000002 rpy=-6.842277657836021e-49 -3.4512664603419266e-31 -1.3877787807814457e-17, axis 1.0 0.0 0.0
- added joint arm_gripper: type continuous, parent STS3215_03a-v1-4, child Moving_Jaw_08d-v1, origin xyz=-0.032799999999999996 -0.023912249999999986 0.027026410000000018 rpy=-1.5707963267948968 3.944304526105059e-31 -1.9721522630525295e-31, axis -2.74128770133849e-31 -0.9063079999999999 -0.422618
- added joint arm_shoulder_lift: type continuous, parent STS3215_03a-v1-1, child SO_ARM100_08k_116_Square-v1, origin xyz=0.0346 0.010249999999999987 -0.032799999999999975 rpy=3.141592653589793 1.7181275903033976e-32 -3.1373434374976504e-48, axis 1.0 0.0 0.0
- added joint arm_shoulder_pan: type continuous, parent STS3215_03a-v1, child Rotation_Pitch_08i-v1, origin xyz=-0.010250000000000084 0.03459999999999999 -0.032799999999999996 rpy=1.5707963267948966 -2.781046729970605e-32 3.94430452610506e-31, axis -3.944304526105059e-31 3.944304526105059e-31 1.0
- added joint arm_wrist_flex: type continuous, parent STS3215_03a-v1-3, child Wrist_Roll_Pitch_08i-v1, origin xyz=0.0346 -0.03408158 0.004398620000000015 rpy=3.1415926535897922 9.860761315262648e-32 -9.503163413661107e-47, axis 1.0 0.0 9.860761315262648e-32
- added joint arm_wrist_roll: type continuous, parent STS3215_03a_Wrist_Roll-v1, child Wrist_Roll_08c-v1, origin xyz=-0.028999999999999998 0.00810632 0.006869499999999995 rpy=3.141592653589793 -0.0 0.0, axis 0.0 0.42261799999999994 -0.9063079999999999
- added joint base_back_wheel: type continuous, parent ST3215_Servo_Motor-v1-2, child omni_wheel_mount-v5-2, origin xyz=0.010249999999999999 -0.035199999999999995 -0.03275 rpy=-1.5707963267948966 1.5707963267948966 0, axis 0.0 0.0 -1.0
- added joint base_left_wheel: type continuous, parent ST3215_Servo_Motor-v1, child omni_wheel_mount-v5, origin xyz=0.010249999999999999 -0.010762340000000004 0.046859090000000006 rpy=-1.5707963267948966 1.5707963267948966 0, axis -0.866025 -2.0578792567370943e-32 0.5
- added joint base_right_wheel: type continuous, parent ST3215_Servo_Motor-v1-1, child omni_wheel_mount-v5-1, origin xyz=0.010249999999999999 0.04636234 -0.014801910000000005 rpy=-1.5707963267948966 1.5707963267948966 0, axis 0.866025 1.0674582272562919e-32 0.5
